File: KiCad/ASR33Old.kicad_pcb (KiCad board)
At the start: 2 copper layers, 45 x 38 mm, 45 parts, among them J1 USB-C, J2 DC, J3 Power, J4 RUN, J5 Tx, J6 Rx, Q1 NX7002AK, SW1 SW_Push, U1 FT231XQ, U2 ESP32-WROOM-32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

Commit message: Resistors
Parts:
- R11: value 10M 1% or 0R -> 100k 1% or 0R
- R12: value 3M 1% or NF -> 30k 1% or NF
Changed lines of the file:
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@@
       (effects (font (size 0.5 0.5) (thickness 0.08)))
     )
-    (fp_text value "3M 1% or NF" (at 1.4 -2.2) (layer "F.Fab")
+    (fp_text value "30k 1% or NF" (at 1.4 -2.2) (layer "F.Fab")
       (effects (font (size 0.4 0.4) (thickness 0.08)))
     )
@@
       (effects (font (size 0.5 0.5) (thickness 0.08)))
     )
-    (fp_text value "10M 1% or 0R" (at -1.6 1.5) (layer "F.Fab")
+    (fp_text value "100k 1% or 0R" (at -1.6 1.5) (layer "F.Fab")
       (effects (font (size 0.4 0.4) (thickness 0.08)))
     )
