File: KiCad/ASR33Old.kicad_sch (KiCad schematic)
At the start: 45 parts, among them J1 USB-C, J2 DC, J3 Power, J4 RUN, J5 Tx, J6 Rx, Q1 NX7002AK, SW1 SW_Push, U1 FT231XQ, U2 ESP32-WROOM-32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

Commit message: Tidy schematic
Parts:
- J1: symbol Connector:USB_C_Receptacle_USB2.0 -> RevK:USB-C
- J2: symbol Connector_Generic:Conn_01x02 -> RevK:PowerIn
Connections:
- no-connect marks 21 -> 19
Changed lines of the file:
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@@
   (junction (at 183.515 63.5) (diameter 0) (color 0 0 0 0)
   )
-  (junction (at 170.815 43.18) (diameter 0) (color 0 0 0 0)
-  )
   (junction (at 60.96 129.54) (diameter 0) (color 0 0 0 0)
   )
@@
   (junction (at 180.975 31.75) (diameter 0) (color 0 0 0 0)
   )
-  (junction (at 170.815 40.64) (diameter 0) (color 0 0 0 0)
-  )
   (no_connect (at 80.645 49.53))
-  (no_connect (at 170.815 53.34))
   (no_connect (at 80.645 41.91))
   (no_connect (at 50.165 80.01))
@@
   (no_connect (at 50.165 72.39))
   (no_connect (at 81.28 165.1))
-  (no_connect (at 170.815 55.88))
   (no_connect (at 50.165 77.47))
   (no_connect (at 50.165 41.91))
@@
     (stroke (width 0) (type default) (color 0 0 0 0))
   )
-  (wire (pts (xy 170.815 38.1) (xy 170.815 40.64))
-    (stroke (width 0) (type default) (color 0 0 0 0))
-  )
   (wire (pts (xy 177.8 63.5) (xy 183.515 63.5))
     (stroke (width 0) (type default) (color 0 0 0 0))
@@
   )
   (wire (pts (xy 245.11 121.285) (xy 259.08 121.285))
-    (stroke (width 0) (type default) (color 0 0 0 0))
-  )
-  (wire (pts (xy 170.815 45.72) (xy 170.815 43.18))
     (stroke (width 0) (type default) (color 0 0 0 0))
   )
@@
     (pin "2")
   )
-  (symbol (lib_id "Connector:USB_C_Receptacle_USB2.0") (at 155.575 40.64 0) (unit 1)
+  (symbol (lib_id "RevK:USB-C") (at 155.575 40.64 0) (unit 1)
     (in_bom yes) (on_board yes)
     (property "Reference" "J1" (id 0) (at 158.2928 18.6182 0))
     (property "Value" "USB-C" (id 1) (at 158.2928 20.9296 0))
-    (property "Footprint" "RevK:USC16-TR-Round" (id 2) (at 159.385 40.64 0)
-      (effects (font (size 1.27 1.27)) hide)
-    )
-    (property "Datasheet" "https://www.usb.org/sites/default/files/documents/usb_type-c.zip" (id 3) (at 159.385 40.64 0)
+    (property "Footprint" "RevK:USC16-TR-Round" (id 2) (at 155.575 20.32 0)
+      (effects (font (size 1.27 1.27)) hide)
+    )
+    (property "Datasheet" "https://www.usb.org/sites/default/files/documents/usb_type-c.zip" (id 3) (at 155.575 17.78 0)
       (effects (font (size 1.27 1.27)) hide)
     )
@@
     )
   )
-  (symbol (lib_id "Connector_Generic:Conn_01x02") (at 264.16 74.93 0) (mirror x) (unit 1)
+  (symbol (lib_id "RevK:PowerIn") (at 264.16 74.93 0) (mirror x) (unit 1)
     (in_bom yes) (on_board yes)
     (property "Reference" "J2" (id 0) (at 262.89 67.31 0)
@@
       (effects (font (size 1.27 1.27)) (justify left))
     )
-    (property "Footprint" "RevK:Molex_MiniSPOX_H2RA" (id 2) (at 264.16 74.93 0)
-      (effects (font (size 1.27 1.27)) hide)
-    )
+    (property "Footprint" "RevK:Molex_MiniSPOX_H2RA" (id 2) (at 264.16 80.01 0)
+      (effects (font (size 1.27 1.27)) hide)
+    )

Commit message: Resistors
Parts:
- R11: value 10M 1% or 0R -> 100k 1% or 0R
- R12: value 3M 1% or NF -> 30k 1% or NF
Changed lines of the file:
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@@
       (effects (font (size 1.27 1.27)) (justify right))
     )
-    (property "Value" "3M 1% or NF" (id 1) (at 233.68 42.545 0)
+    (property "Value" "30k 1% or NF" (id 1) (at 233.68 42.545 0)
       (effects (font (size 1.27 1.27)) (justify right))
     )
@@
       (effects (font (size 1.27 1.27)) (justify left))
     )
-    (property "Value" "10M 1% or 0R" (id 1) (at 228.6 41.91 90)
+    (property "Value" "100k 1% or 0R" (id 1) (at 228.6 41.91 90)
       (effects (font (size 1.27 1.27)) (justify left))
     )
@@
     )
     (path "/fc3ca677-79f2-42b6-a5b3-ff3b18df1d6c"
-      (reference "R11") (unit 1) (value "10M 1% or 0R") (footprint "RevK:R_0603")
+      (reference "R11") (unit 1) (value "100k 1% or 0R") (footprint "RevK:R_0603")
     )
     (path "/83151023-5106-4495-aeff-aefc75dfd6c0"
-      (reference "R12") (unit 1) (value "3M 1% or NF") (footprint "RevK:R_0603")
+      (reference "R12") (unit 1) (value "30k 1% or NF") (footprint "RevK:R_0603")
     )
     (path "/49c7cb3f-a658-4999-a305-f40b4dfcb82f"
