File: PCB/ASR33.kicad_pcb (KiCad board)
At the start: 2 copper layers, 45 x 27 mm, 44 parts, among them J1 Shelly, J2 DC, J3 Power, J4 RUN, J5 Tx, J6 Rx, J7 USB-C, Q1 NX7002AK, SW1 SW_Push, U1 ESP32-PICO-MINI-02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

Commit message: Prog header
Routing:
- net GND: track 46.8 -> 44.7 mm
- net VBUS: track 14.3 -> 12.8 mm
- net Net-(J6-Pin_1): track 10.00 -> 9.12 mm
- net GPIO0: track 51.3 -> 50.6 mm
- net RUN: track 10.4 -> 9.83 mm
- net Net-(C2-Pad1): track 26.2 -> 25.7 mm
