File: PCB/ASR33.kicad_pcb (KiCad board)
At the start: 2 copper layers, 45 x 27 mm, 44 parts, among them J1 Shelly, J2 DC, J3 Power, J4 RUN, J5 Tx, J6 Rx, J7 USB-C, Q1 NX7002AK, SW1 SW_Push, U1 ESP32-PICO-MINI-02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

Commit message: Tidy silk
Parts:
- Q1: footprint Package_TO_SOT_SMD:SOT-23 -> RevK:SOT-23
- U5: footprint Package_SO:SO-4_4.4x3.6mm_P2.54mm -> RevK:SO-4_4.4x3.6mm_P2.54mm
