File: PCB/ASR33WAGO/ASR33.kicad_sch (KiCad schematic)
At the start: 41 parts, among them J1 Tx, J2 Rx, J3 Run, J4 Pwr, J5 Mtr, J6 Reset, J7 USB-C-Socket-V, J8 TC2030-USB-NL-DS, J9 DC, Q1 NX7002AK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

Commit message: PCB Update
Parts:
- C1: LCSC Part # C194427 -> (none); MPN (none) -> C194427
- C8: LCSC Part # C1691 -> (none); MPN (none) -> C1691
- D1: LCSC Part # C1884542 -> (none); MPN (none) -> C1884542
- D2, D3, D6, D7: LCSC Part # C5137770 -> (none); MPN (none) -> C5137770
- D4: LCSC Part # C5349953 -> (none); MPN (none) -> C5349953
- J1, J2: LCSC Part # C2765056 -> (none); MPN (none) -> C2765056
- J3, J4, J5, J9: LCSC Part # C2765055 -> (none); MPN (none) -> C2765055
- J7: LCSC Part # C709357 -> (none); MPN (none) -> C709357
- Q1: JLCPCB Rotation Offset 180 -> (none)
- R1: LCSC Part # C138062 -> (none); MPN (none) -> C138062
- U1: LCSC Part # C2684786 -> (none); MPN (none) -> C2684786; Rotation Offset 180 -> (none)
- U3, U4: LCSC Part # C458148 -> (none); MPN (none) -> C458148; Rotation Offset -90 -> (none)
- U5: Rotation Offset -90 -> (none)
- U8: LCSC Part # C3013941 -> (none); MPN (none) -> C3013941
Changed lines of the file:
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@@
 			)
 		)
-		(property "LCSC Part #" "C709357"
+		(property "MPN" "C709357"
 			(at 155.575 40.64 0)
 			(effects
@@
 			)
 		)
-		(property "LCSC Part #" "C5137770"
+		(property "MPN" "C5137770"
 			(at 122.555 167.64 0)
 			(effects
@@
 			)
 		)
-		(property "LCSC Part #" "C138062"
+		(property "MPN" "C138062"
 			(at 256.54 37.465 0)
 			(effects
@@
 			)
 		)
-		(property "LCSC Part #" "C2765055"
+		(property "MPN" "C2765055"
 			(at 140.97 156.21 0)
 			(effects
@@
 			)
 		)
-		(property "LCSC Part #" "C5349953"
+		(property "MPN" "C5349953"
 			(at 96.52 62.23 0)
 			(effects
@@
 			)
 		)
-		(property "LCSC Part #" "C2765056"
+		(property "MPN" "C2765056"
 			(at 264.16 139.7 0)
 			(effects
@@
 			)
 		)
-		(property "Sim.Enable" "0"
-			(at 266.7 177.165 0)
-			(effects
-				(font
-					(size 1.27 1.27)
-				)
-				(hide yes)
-			)
-		)
 		(instances
 			(project "ASR33"
@@
 			)
 		)
-		(property "Rotation Offset" "-90"
-			(at 229.87 139.7 0)
-			(effects
-				(font
-					(size 1.27 1.27)
-				)
-				(hide yes)
-			)
-		)
 		(pin "1"
 		)
@@
 			)
 		)
-		(property "JLCPCB Rotation Offset" "180"
-			(at 226.695 116.205 0)
-			(effects
-				(font
-					(size 1.27 1.27)
-				)
-				(hide yes)
-			)
-		)
 		(pin "1"
 		)
@@
 			)
 		)
-		(property "LCSC Part #" "C5137770"
+		(property "MPN" "C5137770"
 			(at 118.745 61.595 0)
 			(effects
@@
 			)
 		)
-		(property "LCSC Part #" "C2765055"
+		(property "MPN" "C2765055"
 			(at 140.335 112.395 0)
 			(effects
@@
 			)
 		)
-		(property "LCSC Part #" "C194427"
+		(property "MPN" "C194427"
 			(at 256.54 31.75 0)
 			(effects
@@
 			)
 		)
-		(property "LCSC Part #" "C2765055"
+		(property "MPN" "C2765055"
 			(at 140.97 177.165 0)
 			(effects
@@
 			)
 		)
-		(property "LCSC Part #" "C1884542"
+		(property "MPN" "C1884542"
 			(at 194.945 25.4 0)
 			(effects
@@
 			)
 		)
-		(property "LCSC Part #" "C5137770"
+		(property "MPN" "C5137770"
 			(at 122.555 149.225 0)
 			(effects
@@
 			)
 		)
-		(property "Sim.Enable" "0"
-			(at 269.875 173.99 0)
-			(effects
-				(font
-					(size 1.27 1.27)
-				)
-				(hide yes)
-			)
-		)
 		(instances
 			(project "ASR33"
@@
 			)
 		)
-		(property "LCSC Part #" "C5137770"
+		(property "MPN" "C5137770"
 			(at 128.27 126.365 0)
 			(effects
@@
 			)
 		)
-		(property "Sim.Enable" "0"
-			(at 263.525 173.99 0)
-			(effects
-				(font
-					(size 1.27 1.27)
-				)
-				(hide yes)
-			)
-		)
 		(instances
 			(project "ASR33"
@@
 			)
 		)
-		(property "LCSC Part #" "C2684786"
+		(property "MPN" "C2684786"
 			(at 235.585 64.77 0)
 			(effects
@@
 			)
 		)
-		(property "Rotation Offset" "180"
-			(at 235.585 38.1 0)
-			(effects
-				(font
-					(size 1.27 1.27)
-				)
-				(hide yes)
-			)
-		)
 		(pin "1"
 		)
@@
 			)
 		)
-		(property "Sim.Enable" "0"
-			(at 266.7 170.815 0)
-			(effects
-				(font
-					(size 1.27 1.27)
-				)
-				(hide yes)
-			)
-		)
 		(instances
 			(project "ASR33"
@@
 			)
 		)
-		(property "LCSC Part #" "C2765056"
+		(property "MPN" "C2765056"
 			(at 264.16 121.285 0)
 			(effects
@@
 			)
 		)
-		(property "LCSC Part #" "C458148"
-			(at 170.18 111.76 0)
-			(effects
-				(font
-					(size 1.27 1.27)
-				)
-				(hide yes)
-			)
-		)
-		(property "Rotation Offset" "-90"
+		(property "MPN" "C458148"
 			(at 170.18 111.76 0)
 			(effects
@@
 			)
 		)
-		(property "LCSC Part #" "C3013941"
+		(property "MPN" "C3013941"
 			(at 62.23 107.95 0)
 			(effects
@@
 			)
 		)
-		(property "LCSC Part #" "C2765055"
+		(property "MPN" "C2765055"
 			(at 140.97 133.35 0)
 			(effects
@@
 			)
 		)
-		(property "LCSC Part #" "C1691"
+		(property "MPN" "C1691"
 			(at 256.54 33.655 0)
 			(effects
@@
 			)
 		)
-		(property "LCSC Part #" "C458148"
-			(at 170.18 142.24 0)
-			(effects
-				(font
-					(size 1.27 1.27)
-				)
-				(hide yes)
-			)
-		)
-		(property "Rotation Offset" "-90"
+		(property "MPN" "C458148"
 			(at 170.18 142.24 0)
 			(effects
