File: PCB/ASR33/ASR33.kicad_pcb (KiCad board)
At the start: 2 copper layers, 70 x 70 mm, 40 parts, among them J2 DC, J3 Power, J4 RUN, J5 Tx, J6 Rx, J7 USB-C-Socket-V, J8 Shelly, Q1 NX7002AK, SW1 SW_Push, U1 MD8942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

Commit message: Tweaks
Parts:
- J8: value Shelly -> TC2030-USB-NL-DS; footprint RevK:Shelly -> RevK:Tag-Connect_TC2030-IDC-NL_2x03_P1.27mm_Vertical
- moved J8 7.95 mm to (95.1, 92.0), turned to 0 degrees
- moved J7 1.39 mm to (81.9, 95.1)
- moved R7 0.30 mm to (85.1, 93.3)
- moved R8 0.20 mm to (85.1, 97.2)
Connections:
- J8 pad 1: GND -> VBUS
- J8 pad 2: Net-(J8-0) -> VBUS
- J8 pad 3: +3V3 -> D-
- J8 pad 4: Net-(J8-Rx) -> D+
- J8 pad 5: Net-(J8-Tx) -> GND
- U8 pad 39: Net-(J8-Tx) -> unconnected-(U8-GPIO43-Pad39)
- U8 pad 4: Net-(J8-0) -> unconnected-(U8-GPIO0-Pad4)
- U8 pad 40: Net-(J8-Rx) -> unconnected-(U8-GPIO44-Pad40)
Routing:
- net VBUS: track 14.9 -> 27.3 mm
- net Net-(J8-Rx): track 10.3 -> 0.00 mm
- net Net-(J8-0): track 9.84 -> 0.00 mm
- net Net-(J8-Tx): track 6.57 -> 0.00 mm
- net D-: track 20.9 -> 25.7 mm
- net D+: track 21.5 -> 24.0 mm
- net Net-(J6-Pin_1): track 10.9 -> 12.3 mm
- net Net-(J6-Pin_2): track 11.6 -> 12.9 mm
- net +3V3: track 54.2 -> 53.3 mm, vias 3 -> 4
- net TX20MA: track 30.8 -> 31.7 mm
- net Net-(J7-CC1): track 1.66 -> 2.44 mm
- net RX20MA: track 9.80 -> 10.3 mm
- net GND: track 9.38 -> 9.31 mm, vias 17 -> 23
Other:
- board text added: "12"
- board text added: "Teletype Controller"
- board text removed: "ASR33 Teletype Controller"
- board text removed: "RGB:12"

Commit message: Tweaks
Parts:
- added REF**: Shadow, RevK:Shadow, F.Cu at (100.0, 100.0)

Commit message: New images
Parts:
- removed REF**: Shadow, RevK:Shadow

Commit message: Image and new tc2030
Connections:
- J8 pad 2: VBUS -> D-
- J8 pad 6: GND -> D-
Routing:
- net D-: track 25.7 -> 29.3 mm
- net GND: track 9.31 -> 12.3 mm, vias 23 -> 22
- net VBUS: track 27.3 -> 28.0 mm
