File: PCB/ASR33/ASR33.kicad_sch (KiCad schematic)
At the start: 40 parts, among them J2 DC, J3 Power, J4 RUN, J5 Tx, J6 Rx, J7 USB-C-Socket-V, J8 Shelly, Q1 NX7002AK, SW1 SW_Push, U10 ESP32-S3-MINI-1, U2 MD8942, U3 NCR402U, U4 NCR402U, U5 LTV-356T, U7 QR

Commit message: Tweaks
Parts:
- removed J8: Shelly, RevK:Shelly, symbol RevK:Shelly
- added J8: TC2030-USB-NL-DS, RevK:Tag-Connect_TC2030-IDC-NL_2x03_P1.27mm_Vertical, symbol RevK:TC2030-USB-NL
Connections:
- net D+: now also J8.4 (D+)
- net D-: now also J8.3 (D-)
- net GND: now also J8.5 (GND), J8.6 (GND)
- net VBUS: now also J8.1 (VBUS), J8.2 (VBUS)
- no-connect marks 30 -> 33
Changed lines of the file:
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@@
 	)
 	(junction
-		(at 77.47 53.975)
-		(diameter 0)
-		(color 0 0 0 0)
-	)
-	(junction
 		(at 187.96 142.24)
 		(diameter 0)
@@
 	)
 	(junction
-		(at 77.47 59.055)
-		(diameter 0)
-		(color 0 0 0 0)
-	)
-	(junction
 		(at 187.96 111.76)
 		(diameter 0)
@@
 	)
 	(no_connect
+		(at 77.47 48.895)
+	)
+	(no_connect
 		(at 46.99 66.675)
 	)
@@
 	)
 	(no_connect
+		(at 77.47 56.515)
+	)
+	(no_connect
 		(at 46.99 48.895)
 	)
@@
 	)
 	(no_connect
+		(at 77.47 51.435)
+	)
+	(no_connect
 		(at 77.47 81.915)
 	)
@@
 		)
 	)
+	(global_label "D-"
+		(shape bidirectional)
+		(at 164.465 80.645 0)
+		(fields_autoplaced yes)
+		(effects
+			(font
+				(size 1.27 1.27)
+			)
+			(justify left)
+		)
+		(property "Intersheetrefs" "${INTERSHEET_REFS}"
+			(at 170.5909 80.645 0)
+			(effects
+				(font
+					(size 1.27 1.27)
+				)
+				(justify left)
+				(hide yes)
+			)
+		)
+	)
 	(global_label "PWR"
 		(shape input)
@@
 		)
 	)
+	(global_label "VBUS"
+		(shape output)
+		(at 164.465 76.835 0)
+		(fields_autoplaced yes)
+		(effects
+			(font
+				(size 1.27 1.27)
+			)
+			(justify left)
+		)
+		(property "Intersheetrefs" "${INTERSHEET_REFS}"
+			(at 171.6946 76.835 0)
+			(effects
+				(font
+					(size 1.27 1.27)
+				)
+				(justify left)
+				(hide yes)
+			)
+		)
+	)
 	(global_label "DC"
 		(shape input)
@@
 		)
 	)
+	(global_label "D+"
+		(shape bidirectional)
+		(at 164.465 83.185 0)
+		(fields_autoplaced yes)
+		(effects
+			(font
+				(size 1.27 1.27)
+			)
+			(justify left)
+		)
+		(property "Intersheetrefs" "${INTERSHEET_REFS}"
+			(at 170.5909 83.185 0)
+			(effects
+				(font
+					(size 1.27 1.27)
+				)
+				(justify left)
+				(hide yes)
+			)
+		)
+	)
 	(global_label "BUTTON"
 		(shape input)
@@
 	)
 	(symbol
+		(lib_id "RevK:TC2030-USB-NL")
+		(at 156.845 81.915 0)
+		(unit 1)
+		(exclude_from_sim no)
+		(in_bom no)
+		(on_board yes)
+		(dnp no)
+		(fields_autoplaced yes)
+		(property "Reference" "J8"
+			(at 156.845 70.1505 0)
+			(effects
+				(font
+					(size 1.27 1.27)
+				)
+			)
+		)
+		(property "Value" "TC2030-USB-NL-DS"
+			(at 156.845 72.5748 0)
+			(effects
+				(font
+					(size 1.27 1.27)
+				)
+			)
+		)
+		(property "Footprint" "RevK:Tag-Connect_TC2030-IDC-NL_2x03_P1.27mm_Vertical"
+			(at 156.591 91.059 0)
+			(effects
+				(font
+					(size 1.27 1.27)
+				)
+				(hide yes)
+			)
+		)
+		(property "Datasheet" " ~"
+			(at 160.655 83.185 0)
+			(effects
+				(font
+					(size 1.27 1.27)
+				)
+				(hide yes)
+			)
+		)
+		(property "Description" "TC2030-USB-NL"
+			(at 156.845 69.215 0)
+			(effects
+				(font
+					(size 1.27 1.27)
+				)
+				(hide yes)
+			)
+		)
+		(pin "1"
+		)
+		(pin "2"
+		)
+		(pin "3"
+		)
+		(pin "4"
+		)
+		(pin "5"
+		)
+		(pin "6"
+		)
+		(instances
+			(project "ASR33"
+				(path "/46c350bb-7de4-4e81-aafd-4af55e37aab0"
+					(reference "J8")
+					(unit 1)
+				)
+			)
+		)
+	)
+	(symbol
 		(lib_id "RevK:Hidden")
 		(at 256.54 43.18 90)
@@
 	)
 	(symbol
+		(lib_id "power:GND")
+		(at 164.465 86.995 90)
+		(unit 1)
+		(exclude_from_sim no)
+		(in_bom yes)
+		(on_board yes)
+		(dnp no)
+		(fields_autoplaced yes)
+		(property "Reference" "#PWR012"
+			(at 170.815 86.995 0)
+			(effects
+				(font
+					(size 1.27 1.27)
+				)
+				(hide yes)
+			)
+		)
+		(property "Value" "GND"
+			(at 167.64 86.995 90)
+			(effects
+				(font
+					(size 1.27 1.27)
+				)
+				(justify right)
+			)
+		)
+		(property "Footprint" ""
+			(at 164.465 86.995 0)
+			(effects
+				(font
+					(size 1.27 1.27)
+				)
+				(hide yes)
+			)
+		)
+		(property "Datasheet" ""
+			(at 164.465 86.995 0)
+			(effects
+				(font
+					(size 1.27 1.27)
+				)
+				(hide yes)
+			)
+		)
+		(property "Description" "Power symbol creates a global label with name \"GND\" , ground"
+			(at 164.465 86.995 0)
+			(effects
+				(font
+					(size 1.27 1.27)
+				)
+				(hide yes)
+			)
+		)
+		(pin "1"
+		)
+		(instances
+			(project "ASR33"
+				(path "/46c350bb-7de4-4e81-aafd-4af55e37aab0"
+					(reference "#PWR012")
+					(unit 1)
+				)
+			)
+		)
+	)
+	(symbol
 		(lib_id "RevK:VCUT")
 		(at 263.525 173.99 90)
@@
 					(unit 1)
 				)
-			)
-		)
-	)
-	(symbol
-		(lib_id "RevK:Shelly")
-		(at 77.47 53.975 0)
-		(unit 1)
-		(exclude_from_sim no)
-		(in_bom no)
-		(on_board yes)
-		(dnp no)
-		(property "Reference" "J8"
-			(at 76.2 45.72 0)
-			(effects
-				(font
-					(size 1.27 1.27)
-				)
-				(justify left)
-			)
-		)
-		(property "Value" "Shelly"
-			(at 79.375 45.72 0)
-			(effects
-				(font
-					(size 1.27 1.27)
-				)
-				(justify left)
-			)
-		)
-		(property "Footprint" "RevK:Shelly"
-			(at 80.01 62.23 0)
-			(effects
-				(font
-					(size 1.27 1.27)
-				)
-				(hide yes)
-			)
-		)
-		(property "Datasheet" ""
-			(at 80.01 62.23 0)
-			(effects
-				(font
-					(size 1.27 1.27)
-				)
-				(hide yes)
-			)
-		)
-		(property "Description" ""
-			(at 77.47 53.975 0)
-			(effects
-				(font
-					(size 1.27 1.27)
-				)
-				(hide yes)
-			)
-		)
-		(pin "1"
-		)
-		(pin "2"
-		)
-		(pin "3"
-		)
-		(pin "4"
-		)
-		(pin "5"
-		)
-		(instances
-			(project "Access"
-				(path "/2a267270-6585-45e3-a633-b53049f10066"
-					(reference "J8")
-					(unit 1)
-				)
-			)
-			(project "USBA"
-				(path "/2d210a96-f81f-42a9-8bf4-1b43c11086f3"
-					(reference "J2")
-					(unit 1)
-				)
-			)
-			(project "ASR33"
-				(path "/46c350bb-7de4-4e81-aafd-4af55e37aab0"
-					(reference "J8")
-					(unit 1)
-				)

Commit message: PCB Update
Parts:
- C1: renamed from C21; LCSC Part # C194427 -> (none); MPN (none) -> C194427
- C8: renamed from C22; LCSC Part # C1691 -> (none); MPN (none) -> C1691
- D1: renamed from D3; LCSC Part # C1884542 -> (none); MPN (none) -> C1884542
- D2, D3, D6, D7: LCSC Part # C5137770 -> (none); MPN (none) -> C5137770
- D4: renamed from D1; LCSC Part # C5349953 -> (none); MPN (none) -> C5349953
- J7: LCSC Part # C709357 -> (none); MPN (none) -> C709357
- Q1: JLCPCB Rotation Offset 180 -> (none)
- R1: renamed from R14; LCSC Part # C138062 -> (none); MPN (none) -> C138062
- U1: renamed from U2; LCSC Part # C2684786 -> (none); MPN (none) -> C2684786
- U3, U4, U5: JLCPCB Rotation Offset -90 -> (none)
- U8: renamed from U10; LCSC Part # C3013941 -> (none); MPN (none) -> C3013941
- renumbered C19 to C10, C20 to C11, C23 to C12, C18 to C9, L4 to L2, R26 to R13, R15 to R2, R27 to R3
Changed lines of the file:
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@@
 (kicad_sch
-	(version 20231120)
+	(version 20241209)
 	(generator "eeschema")
-	(generator_version "8.0")
+	(generator_version "9.0")
 	(paper "A4")
 	(title_block
@@
 		(on_board yes)
 		(dnp no)
-		(property "Reference" "#PWR07"
+		(property "Reference" "#PWR04"
 			(at 73.66 53.975 0)
 			(effects
@@
 		(on_board yes)
 		(dnp no)
-		(property "Reference" "C23"
+		(property "Reference" "C12"
 			(at 261.62 35.56 90)
 			(effects
@@
 			)
 		)
-		(property "LCSC Part #" "C709357"
+		(property "MPN" "C709357"
 			(at 155.575 40.64 0)
 			(effects
@@
 		(on_board yes)
 		(dnp no)
-		(property "Reference" "R27"
+		(property "Reference" "R3"
 			(at 257.81 41.275 0)
 			(effects
@@
 		(on_board yes)
 		(dnp no)
-		(property "Reference" "C18"
+		(property "Reference" "C9"
 			(at 50.165 27.797 0)
 			(effects
@@
 			)
 		)
-		(property "LCSC Part #" "C5137770"
+		(property "MPN" "C5137770"
 			(at 122.555 126.365 0)
 			(effects
@@
 		(on_board yes)
 		(dnp no)
-		(property "Reference" "R14"
+		(property "Reference" "R1"
 			(at 259.08 37.465 0)
 			(effects
@@
 			)
 		)
-		(property "LCSC Part #" "C138062"
+		(property "MPN" "C138062"
 			(at 256.54 37.465 0)
 			(effects
@@
 		(dnp no)
 		(fields_autoplaced yes)
-		(property "Reference" "#PWR014"
+		(property "Reference" "#PWR029"
 			(at 59.055 29.21 0)
 			(effects
@@
 		(on_board yes)
 		(dnp no)
-		(property "Reference" "D1"
+		(property "Reference" "D4"
 			(at 95.25 73.66 0)
 			(do_not_autoplace yes)
@@
 			)
 		)
-		(property "LCSC Part #" "C5349953"
+		(property "MPN" "C5349953"
 			(at 96.52 62.23 0)
 			(effects
@@
 		(on_board yes)
 		(dnp no)
-		(property "Reference" "R15"
+		(property "Reference" "R2"
 			(at 259.08 39.37 90)
 			(effects
@@
 			)
 		)
-		(property "JLCPCB Rotation Offset" "-90"
-			(at 229.87 139.7 0)
-			(effects
-				(font
-					(size 1.27 1.27)
-				)
-				(hide yes)
-			)
-		)
 		(pin "1"
 		)
@@
 		(on_board yes)
 		(dnp no)
-		(property "Reference" "L4"
+		(property "Reference" "L2"
 			(at 257.81 43.18 90)
 			(effects
@@
 			)
 		)
-		(property "JLCPCB Rotation Offset" "180"
-			(at 226.695 116.205 0)
-			(effects
-				(font
-					(size 1.27 1.27)
-				)
-				(hide yes)
-			)
-		)
 		(pin "1"
 		)
@@
 		(dnp no)
 		(fields_autoplaced yes)
-		(property "Reference" "#PWR046"
+		(property "Reference" "#PWR039"
 			(at 65.405 39.37 0)
 			(effects
@@
 		(on_board yes)
 		(dnp no)
-		(property "Reference" "#PWR04"
+		(property "Reference" "#PWR03"
 			(at 235.585 53.975 0)
 			(effects
@@
 		(dnp no)
 		(fields_autoplaced yes)
-		(property "Reference" "#PWR022"
+		(property "Reference" "#PWR030"
 			(at 59.055 39.37 0)
 			(effects
@@
 			)
 		)
-		(property "LCSC Part #" "C5137770"
+		(property "MPN" "C5137770"
 			(at 118.745 61.595 0)
 			(effects
@@
 		(on_board yes)
 		(dnp no)
-		(property "Reference" "C21"
+		(property "Reference" "C1"
 			(at 257.81 31.75 0)
 			(effects
@@
 			)
 		)
-		(property "LCSC Part #" "C194427"
+		(property "MPN" "C194427"
 			(at 256.54 31.75 0)
 			(effects
@@
 		(on_board yes)
 		(dnp no)
-		(property "Reference" "D3"
+		(property "Reference" "D1"
 			(at 194.945 19.8882 0)
 			(effects
@@
 			)
 		)
-		(property "LCSC Part #" "C1884542"
+		(property "MPN" "C1884542"
 			(at 194.945 25.4 0)
 			(effects
@@
 		(on_board yes)
 		(dnp no)
-		(property "Reference" "R26"
+		(property "Reference" "R13"
 			(at 92.71 99.06 90)
 			(effects
@@
 		(dnp no)
 		(fields_autoplaced yes)
-		(property "Reference" "#PWR044"
+		(property "Reference" "#PWR033"
 			(at 65.405 29.21 0)
 			(effects
@@
 			)
 		)
-		(property "LCSC Part #" "C5137770"
+		(property "MPN" "C5137770"
 			(at 122.555 149.225 0)
 			(effects
@@
 		(dnp no)
 		(fields_autoplaced yes)
-		(property "Reference" "#PWR063"
+		(property "Reference" "#PWR041"
 			(at 90.805 116.84 0)
 			(effects
@@
 		(dnp no)
 		(fields_autoplaced yes)
-		(property "Reference" "#PWR063"
+		(property "Reference" "#PWR05"
 			(at 83.82 59.055 0)
 			(effects
@@
 			)
 		)
-		(property "LCSC Part #" "C5137770"
+		(property "MPN" "C5137770"
 			(at 128.27 126.365 0)
 			(effects
@@
 		(dnp no)
 		(fields_autoplaced yes)
-		(property "Reference" "#PWR062"
+		(property "Reference" "#PWR040"
 			(at 90.805 99.06 0)
 			(effects
@@
 		(on_board yes)
 		(dnp no)
-		(property "Reference" "U2"
+		(property "Reference" "U1"
 			(at 235.585 31.75 0)
 			(effects
@@
 			)
 		)
-		(property "LCSC Part #" "C2684786"
+		(property "MPN" "C2684786"
 			(at 235.585 64.77 0)
 			(effects
@@
 		(dnp no)
 		(fields_autoplaced yes)
-		(property "Reference" "C19"
+		(property "Reference" "C10"
 			(at 68.326 28.186 0)
 			(effects
@@
 		(dnp no)
 		(fields_autoplaced yes)
-		(property "Reference" "#PWR062"
+		(property "Reference" "#PWR010"
 			(at 95.25 73.66 0)
 			(effects
@@
 		(dnp no)
 		(fields_autoplaced yes)
-		(property "Reference" "#PWR03"
+		(property "Reference" "#PWR02"
 			(at 227.965 38.1 0)
 			(effects
@@
 			)
 		)
-		(property "JLCPCB Rotation Offset" "-90"
-			(at 170.18 111.76 0)
-			(effects
-				(font
-					(size 1.27 1.27)
-				)
-				(hide yes)
-			)
-		)
 		(pin "1"
 		)
@@
 		(dnp no)
 		(fields_autoplaced yes)
-		(property "Reference" "U10"
+		(property "Reference" "U8"
 			(at 62.23 41.7282 0)
 			(effects
@@
 			)
 		)
-		(property "LCSC Part #" "C3013941"
+		(property "MPN" "C3013941"
 			(at 62.23 107.95 0)
 			(effects
@@
 		(on_board yes)
 		(dnp no)
-		(property "Reference" "C22"
+		(property "Reference" "C8"
 			(at 257.81 33.655 0)
 			(effects
@@
 			)
 		)
-		(property "LCSC Part #" "C1691"
+		(property "MPN" "C1691"
 			(at 256.54 33.655 0)
 			(effects
@@
 		(dnp no)
 		(fields_autoplaced yes)
-		(property "Reference" "#PWR063"
+		(property "Reference" "#PWR01"
 			(at 95.25 83.82 0)
 			(effects
@@
 		(dnp no)
 		(fields_autoplaced yes)
-		(property "Reference" "C20"
+		(property "Reference" "C11"
 			(at 93.726 105.8453 0)
 			(effects
@@
 			)
 		)
-		(property "JLCPCB Rotation Offset" "-90"
-			(at 170.18 142.24 0)
-			(effects
-				(font
-					(size 1.27 1.27)
-				)
-				(hide yes)
-			)
-		)
 		(pin "1"
 		)
@@
 		)
 	)
+	(embedded_fonts no)
 )

Commit message: Image and new tc2030
Connections:
- net D-: now also J8.2 (NC), J8.6 (NC)
- net GND: no longer J8.6 (GND)
- net VBUS: no longer J8.2 (VBUS)
Changed lines of the file:
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@@
 			)
 		)
-		(property "Datasheet" " ~"
+		(property "Datasheet" "~"
 			(at 160.655 83.185 0)
 			(effects
